Commit message: add parent and root arg in dragn_link.urdf.xacro

File: robots/dragon/urdf/dragon_link.urdf.xacro (robot description, xacro)
@@ -3,5 +3,5 @@
     xmlns:xacro="http://www.ros.org/wiki/xacro" name="dragon_link" >
   <!-- D-H kai description(different from prof.nakamura) -->
-  <xacro:macro name="dragon_module" params="self child baselink">
+  <xacro:macro name="dragon_module" params="self child:=-1 parent:=-1 root baselink">
     <!-- link -->
     <link name="link${self}">
@@ -172,9 +172,15 @@
     <xacro:damping_factor link ="thrust${self}"/>
     <!-- joint -->
-    <xacro:unless value="${self == child}">
+    <xacro:unless value="${self == child or self == parent}">
       <joint name="joint${self}_pitch" type="revolute">
         <limit effort="10.0" lower="${-pi/2}" upper="${pi/2}" velocity="0.1"/>
-        <parent link="link${self}"/>
-        <child link="inter_joint${self}"/>
+        <xacro:if value="${parent > 0}">
+          <parent link="inter_joint${self}"/>
+          <child link="link${self}"/>
+        </xacro:if>
+        <xacro:if value="${child > 0}">
+          <parent link="link${self}"/>
+          <child link="inter_joint${self}"/>
+        </xacro:if>
         <origin rpy="0 0 0" xyz="${link_length} 0 0"/>
         <axis xyz="0 1 0"/>
@@ -200,6 +206,12 @@
       <joint name="joint${self}_yaw" type="revolute">
         <limit effort="10.0" lower="${-pi/2}" upper="${pi/2}" velocity="0.1"/>
-        <parent link="inter_joint${self}"/>
-        <child link="link${child}"/>
+        <xacro:if value="${child > 0}">
+          <parent link="inter_joint${self}"/>
+          <child link="link${child}"/>
+        </xacro:if>
+        <xacro:if value="${parent > 0}">
+          <parent link="link${parent}"/>
+          <child link="inter_joint${self}"/>
+        </xacro:if>
         <origin rpy="0 0 0" xyz="${2 * inter_joint_x_offset} 0 0"/>
         <axis xyz="0 0 1"/>
@@ -211,5 +223,5 @@
       </gazebo>
     </xacro:unless>
-    <xacro:if value="${self == 1}">
+    <xacro:if value="${root}">
       <!-- dummy root link for KDL -->
       <link name="root">
@@ -250,5 +262,5 @@
     </xacro:if>
     <!-- hardware interface -->
-    <xacro:unless value="${self == child}">
+    <xacro:if value="${self != child and self != parent}">
       <transmission name="joint${self}_pitch_tran">
         <type>transmission_interface/SimpleTransmission</type>
@@ -275,5 +287,5 @@
         </actuator>
       </transmission>
-    </xacro:unless>
+    </xacro:if>
     <transmission name="gimbal${self}_roll_tran">
       <type>transmission_interface/SimpleTransmission</type>

Commit message: fix dragon_link.urdf.xacro for head

File: robots/dragon/urdf/dragon_link.urdf.xacro (robot description, xacro)
@@ -56,4 +56,27 @@
     </link>
     <xacro:damping_factor link ="link${self}"/>
+    <link name="link${self}_edge">
+      <inertial>
+        <origin xyz="0 0 0" rpy="0 0 0"/>
+        <mass value="0.00001"/>
+        <inertia
+            ixx="0.000001" ixy="0.0" ixz="0.0"
+            iyy="0.000001" iyz="0.0"
+            izz="0.000002"/>
+      </inertial>
+    </link>
+    <joint name="link${self}_edge_fixed_joint" type="fixed">
+      <xacro:if value="${child > 0}">
+        <parent link="link${self}"/>
+        <child link="link${self}_edge"/>
+        <origin rpy="0 0 0" xyz="${link_length} 0 0"/>
+      </xacro:if>
+      <xacro:if value="${parent > 0}">
+        <parent link="link${self}_edge"/>
+        <child link="link${self}"/>
+        <origin rpy="0 0 0" xyz="${-1 * link_length} 0 0 "/>
+      </xacro:if>
+      <axis xyz="0 0 1"/>
+    </joint>
     <!-- gimbal roll -->
     <joint name="gimbal${self}_roll" type="revolute">
@@ -175,14 +198,16 @@
       <joint name="joint${self}_pitch" type="revolute">
         <limit effort="10.0" lower="${-pi/2}" upper="${pi/2}" velocity="0.1"/>
+        <xacro:if value="${child > 0}">
+          <parent link="link${self}_edge"/>
+          <child link="inter_joint${self}"/>
+          <origin rpy="0 0 0" xyz="0 0 0"/>
+          <axis xyz="0 1 0"/>
+        </xacro:if>
         <xacro:if value="${parent > 0}">
           <parent link="inter_joint${self}"/>
-          <child link="link${self}"/>
-        </xacro:if>
-        <xacro:if value="${child > 0}">
-          <parent link="link${self}"/>
-          <child link="inter_joint${self}"/>
-        </xacro:if>
-        <origin rpy="0 0 0" xyz="${link_length} 0 0"/>
-        <axis xyz="0 1 0"/>
+          <child link="link${self}_edge"/>
+          <origin rpy="0 0 0" xyz="${-2 * inter_joint_x_offset} 0 0"/>
+          <axis xyz="0 -1 0"/>
+        </xacro:if>
         <dynamics damping="0.9" friction="0.05"/>
       </joint>
@@ -198,5 +223,10 @@
         </inertial>
         <visual>
-          <origin rpy="0 0 0" xyz="${inter_joint_x_offset} 0 0"/>
+          <xacro:if value="${child > 0}">
+            <origin rpy="0 0 0" xyz="${inter_joint_x_offset} 0 0"/>
+          </xacro:if>
+          <xacro:if value="${parent > 0}">
+            <origin rpy="0 0 0" xyz="${-1 * inter_joint_x_offset} 0 0"/>
+          </xacro:if>
           <geometry>
             <mesh filename="package://dragon/urdf/mesh/inter_joint_junction.dae"/>
@@ -209,11 +239,13 @@
           <parent link="inter_joint${self}"/>
           <child link="link${child}"/>
+          <origin rpy="0 0 0" xyz="${2 * inter_joint_x_offset} 0 0"/>
+          <axis xyz="0 0 1"/>
         </xacro:if>
         <xacro:if value="${parent > 0}">
           <parent link="link${parent}"/>
           <child link="inter_joint${self}"/>
-        </xacro:if>
-        <origin rpy="0 0 0" xyz="${2 * inter_joint_x_offset} 0 0"/>
-        <axis xyz="0 0 1"/>
+          <origin rpy="0 0 0" xyz="0 0 0"/>
+          <axis xyz="0 0 -1"/>
+        </xacro:if>
         <dynamics damping="0.9" friction="0.05"/>
       </joint>
